File: bq76920.sch (KiCad schematic (older format))
At the start: 64 parts, among them P3 ON/OFF, Q1 DMN2004K, Q2 BSS84, Q3 DMN2004K, Q4 2N7002, Q5 DMN2004K, Q6 DMN2004K, Q7 DMN2004K, SW1 SW_PUSH, U1 BQ76920

Commit message: Small fixes for final gerber export (DRU check passed)
Parts:
- Q2: symbol Q_NMOS_GSD -> Q_PMOS_GSD
Changed lines of the file:
@@
 encoding utf-8
 Sheet 2 6
-Title ""
-Date ""
-Rev ""
-Comp ""
-Comment1 ""
-Comment2 ""
+Title "Libre Solar BMS 5s"
+Date "2017-05-27"
+Rev "0.1"
+Comp "Libre Solar (http://libre.solar)"
+Comment1 "License: CC-BY-SA"
+Comment2 "Author: Martin Jäger"
 Comment3 ""
 Comment4 ""
@@
 BQ_ALERT
 $Comp
-L Q_NMOS_GSD Q2
+L Q_PMOS_GSD Q2
 U 1 1 58E3A897
 P 9000 1600
