File: interfaces.sch (KiCad schematic (older format))
At the start: 19 parts, among them J4 UEXT, J6 Screw_Terminal_1x02, P2 USB_B, P3 USB_OTG, U8 TJA1042T/3

Commit message: Small fixes for final gerber export (DRU check passed)
Parts:
- removed J6: Screw_Terminal_1x02, Connectors_Terminal_Blocks:TerminalBlock_Pheonix_MKDS1.5-2pol, symbol Screw_Terminal_1x02
- removed P2: USB_B, Connectors:USB_B, symbol USB_B
- removed R31, R32: 0, Resistors_SMD:R_0603, symbol R
- added RT1: 200mA, LibreSolar:R_1206_3216, symbol R_PTC
- C24: renamed from C26; footprint Capacitors_SMD:C_0603 -> LibreSolar:C_0603_1608; MFR Murata -> (none); MPN GRM188R71H104KA93D -> (none); Manufacturer (none) -> Murata; PartNumber (none) -> GRM188R71H104KA93D
- C25: renamed from C39; footprint Capacitors_SMD:C_0603 -> LibreSolar:C_0603_1608; MFR Murata -> (none); MPN GRM188R71H104KA93D -> (none); Manufacturer (none) -> Murata; PartNumber (none) -> GRM188R71H104KA93D
- C26: renamed from C25; footprint Capacitors_SMD:C_0603 -> LibreSolar:C_0603_1608; MFR Murata -> (none); MPN GRM188R71H104KA93D -> (none); Manufacturer (none) -> Murata; PartNumber (none) -> GRM188R71H104KA93D; SPN - -> (none); SPR - -> (none); SPURL - -> (none)
- D15: renamed from D3; Alternative (none) -> WE-TVS 82400102; MFR STMicroelectronics -> (none); MPN USBLC6-2SC6 -> (none); Manufacturer (none) -> STMicroelectronics; PartNumber (none) -> USBLC6-2SC6
- D16: renamed from D4; footprint TO_SOT_Packages_SMD:SOT-23 -> LibreSolar:SOT-23; MFR ON Semiconductor -> (none); MPN NUP2105LT1G -> (none); Manufacturer (none) -> ON Semiconductor; PartNumber (none) -> NUP2105LT1G
- J2: renamed from J4; footprint Pin_Headers:Pin_Header_Straight_2x05_Pitch2.54mm -> LibreSolar:Box_Header_2x05x2.54mm_Straight; Manufacturer (none) -> Würth; PartNumber (none) -> 61201021621
- JP1: renamed from JP3; footprint Pin_Headers:Pin_Header_Straight_1x02_Pitch2.54mm -> Pin_Headers:Pin_Header_Angled_2x01_Pitch2.54mm
- JP2: renamed from JP1; footprint Connectors:RJ45_8 -> LibreSolar:RJ45_8P8C; MFR Amphenol FCI -> (none); MPN 54602-908LF -> (none); Manufacturer (none) -> FCI / Amphenol; PartNumber (none) -> 54602-908LF
- JP3: renamed from JP2; footprint Connectors:RJ45_8 -> LibreSolar:RJ45_8P8C; MFR Amphenol FCI -> (none); MPN 54602-908LF -> (none); Manufacturer (none) -> FCI / Amphenol; PartNumber (none) -> 54602-908LF
- P4: renamed from P3; value USB_OTG -> USB_Micro-B; footprint LibreSolar:Wuerth_USB_Micro_USB_vert_Type_B_614105150721 -> LibreSolar:USB_Micro-B_10103594-0001LF; MFR Wuerth -> (none); MPN 614105150721 -> (none); Manufacturer (none) -> FCI; PartNumber (none) -> 10103594-0001LF; SPR Mouser -> (none)
- R31: renamed from R46; footprint Resistors_SMD:R_0603 -> LibreSolar:R_0603_1608; MFR Yageo -> (none); MPN RC0603FR-07100KL -> (none); Manufacturer (none) -> Yageo; PartNumber (none) -> RC0603FR-07100KL
- R32: renamed from R36; footprint Resistors_SMD:R_1206 -> LibreSolar:R_1206_3216; MFR Yageo -> (none); MPN RC1206FR-07120RL -> (none); Manufacturer (none) -> Yageo; PartNumber (none) -> RC1206FR-07120RL
- R33: renamed from R34; footprint Resistors_SMD:R_0603 -> LibreSolar:R_0603_1608; MFR Yageo -> (none); MPN RC0603FR-072K2L -> (none); Manufacturer (none) -> Yageo; PartNumber (none) -> RC0603FR-072K2L
- R34: renamed from R35; footprint Resistors_SMD:R_0603 -> LibreSolar:R_0603_1608; MFR Yageo -> (none); MPN RC0603FR-072K2L -> (none); Manufacturer (none) -> Yageo; PartNumber (none) -> RC0603FR-072K2L
- U4: renamed from U8; MFR NXP -> (none); MPN TJA1042T/3/1J -> (none); Manufacturer (none) -> NXP; PartNumber (none) -> TJA1042T/3/1J; SPR Mouser -> (none)
Connections:
- net labels added: RJ45_P4, RJ45_P5
- net labels removed: USB_SH
- wire segments 87 -> 76
- no-connect marks 7 -> 0
Other:
- note removed: "Alt. to USBLC6-2:\nWE-TVS 82400102\n\nTwo alternative connectors\n(old type B and Micro type B)\nWürth 614105150721"
- moved on the sheet: C24, C25, C26, D15, D16, J2, JP1, JP2, JP3, P4, R31, R32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
