File: power-pcb/Switch-N-Sense.sch (KiCad schematic (older format))
At the start: 40 parts, among them P1 CONN_01X01, P2 CONN_01X01, P3 CONN_01X01, P4 CONN_01X01, P5 CONN_01X01, P6 Conn_Switch-N-Sense, Q1 CSD18540Q5B, Q2 CSD18540Q5B, Q3 CSD18540Q5B, Q4 CSD18540Q5B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

Commit message: Issue #6 fixed
Parts:
- added R17: 1M, LibreSolar:R_0603_1608, symbol R
- D1, D2: value SMCJ36A -> SMCJ24A; PartNumber SMCJ36A -> SMCJ24A
- Q1, Q2, Q3, Q4: value CSD18540Q5B -> BSC010N04LS; Manufacturer Texas Instruments -> Infineon; PartNumber CSD18540Q5B -> BSC010N04LS
- Q5: symbol Q_PMOS_GDS -> Q_PMOS_GSD
Connections:
- net LOAD+: now also Q5.3 (D); no longer Q5.2 (D)
- net PCHG_G: now also R17.2
- net at R5.1, R6.1, R7.1: now also Q5.2 (S), R17.1; no longer Q5.3 (S)
Other:
- note added: "Maximum voltage: 24 V\n(--> only suitable for up to 5 Li-Ion / Li Polymer cells)\nMaximum current: 50 A continuous, 100 A peak"
- note removed: "Maximum voltage: 36 V\n(--> only suitable for up to 8 LiFePO4 cells)\nMaximum current: 50 A continuous, 100 A peak"
Changed lines of the file:
@@
 P 3000 2700
 F 0 "Q1" V 2950 2450 50  0000 L CNN
-F 1 "CSD18540Q5B" V 3250 2550 50  0000 L CNN
+F 1 "BSC010N04LS" V 3250 2450 50  0000 L CNN
 F 2 "LibreSolar:5X6_MOSFET" H 3200 2800 50  0001 C CNN
 F 3 "" H 3000 2700 50  0000 C CNN
-F 4 "Texas Instruments" H 0   500 60  0001 C CNN "Manufacturer"
-F 5 "CSD18540Q5B" H 0   500 60  0001 C CNN "PartNumber"
+F 4 "Infineon" H 0   500 60  0001 C CNN "Manufacturer"
+F 5 "BSC010N04LS" H 0   500 60  0001 C CNN "PartNumber"
 	1    3000 2700
 	0    1    1    0
@@
 P 3000 3400
 F 0 "Q3" V 2950 3150 50  0000 L CNN
-F 1 "CSD18540Q5B" V 3250 3250 50  0000 L CNN
+F 1 "BSC010N04LS" V 3250 3150 50  0000 L CNN
 F 2 "LibreSolar:5X6_MOSFET" H 3200 3500 50  0001 C CNN
 F 3 "" H 3000 3400 50  0000 C CNN
-F 4 "Texas Instruments" H 0   500 60  0001 C CNN "Manufacturer"
-F 5 "CSD18540Q5B" H 0   500 60  0001 C CNN "PartNumber"
+F 4 "Infineon" H 0   500 60  0001 C CNN "Manufacturer"
+F 5 "BSC010N04LS" H 0   500 60  0001 C CNN "PartNumber"
 	1    3000 3400
 	0    1    1    0
@@
 P 4300 2700
 F 0 "Q2" V 4250 2850 50  0000 L CNN
-F 1 "CSD18540Q5B" V 4550 2550 50  0000 L CNN
+F 1 "BSC010N04LS" V 4550 2500 50  0000 L CNN
 F 2 "LibreSolar:5X6_MOSFET" H 4500 2800 50  0001 C CNN
 F 3 "" H 4300 2700 50  0000 C CNN
-F 4 "Texas Instruments" H 4300 2700 60  0001 C CNN "Manufacturer"
-F 5 "CSD18540Q5B" H 4300 2700 60  0001 C CNN "PartNumber"
+F 4 "Infineon" H 4300 2700 60  0001 C CNN "Manufacturer"
+F 5 "BSC010N04LS" H 4300 2700 60  0001 C CNN "PartNumber"
 	1    4300 2700
 	0    -1   1    0
@@
 P 4300 3400
 F 0 "Q4" V 4250 3550 50  0000 L CNN
-F 1 "CSD18540Q5B" V 4550 3300 50  0000 L CNN
+F 1 "BSC010N04LS" V 4550 3150 50  0000 L CNN
 F 2 "LibreSolar:5X6_MOSFET" H 4500 3500 50  0001 C CNN
 F 3 "" H 4300 3400 50  0000 C CNN
-F 4 "Texas Instruments" H 0   500 60  0001 C CNN "Manufacturer"
-F 5 "CSD18540Q5B" H 0   500 60  0001 C CNN "PartNumber"
+F 4 "Infineon" H 0   500 60  0001 C CNN "Manufacturer"
+F 5 "BSC010N04LS" H 0   500 60  0001 C CNN "PartNumber"
 	1    4300 3400
 	0    -1   1    0
@@
 P 2000 4400
 F 0 "D1" H 2000 4500 50  0000 C CNN
-F 1 "SMCJ36A" H 2000 4300 50  0000 C CNN
+F 1 "SMCJ24A" H 2000 4300 50  0000 C CNN
 F 2 "LibreSolar:D_SMC" V 2000 4400 50  0001 C CNN
 F 3 "" V 2000 4400 50  0000 C CNN
 F 4 "Bourns" H 2000 4400 60  0001 C CNN "Manufacturer"
-F 5 "SMCJ36A" H 2000 4400 60  0001 C CNN "PartNumber"
+F 5 "SMCJ24A" H 2000 4400 60  0001 C CNN "PartNumber"
 	1    2000 4400
 	0    -1   1    0
@@
 P 5400 4500
 F 0 "D2" H 5400 4600 50  0000 C CNN
-F 1 "SMCJ36A" H 5400 4400 50  0000 C CNN
+F 1 "SMCJ24A" H 5400 4400 50  0000 C CNN
 F 2 "LibreSolar:D_SMC" V 5400 4500 50  0001 C CNN
 F 3 "" V 5400 4500 50  0000 C CNN
 F 4 "Bourns" H 5400 4500 60  0001 C CNN "Manufacturer"
-F 5 "SMCJ36A" H 5400 4500 60  0001 C CNN "PartNumber"
+F 5 "SMCJ24A" H 5400 4500 60  0001 C CNN "PartNumber"
 	1    5400 4500
 	0    -1   1    0
@@
 $EndComp
 $Comp
-L Q_PMOS_GDS Q5
+L Q_PMOS_GSD Q5
 U 1 1 58F82D00
 P 5200 1800
@@
 Text Label 5000 2400 2    50   ~ 0
 DSG_G
-Text Label 4800 1500 0    50   ~ 0
+Text Label 4500 1500 0    50   ~ 0
 PCHG_G
 $Comp
@@
 $EndComp
 $Comp
-L GND #PWR01
+L GND #PWR1
 U 1 1 58F8A6D0
 P 7900 3000
-F 0 "#PWR01" H 7900 2750 50  0001 C CNN
+F 0 "#PWR1" H 7900 2750 50  0001 C CNN
 F 1 "GND" H 7900 2850 50  0000 C CNN
 F 2 "" H 7900 3000 50  0000 C CNN
@@
 $EndComp
 $Comp
-L GND #PWR02
+L GND #PWR5
 U 1 1 58F8A862
 P 2200 5400
-F 0 "#PWR02" H 2200 5150 50  0001 C CNN
+F 0 "#PWR5" H 2200 5150 50  0001 C CNN
 F 1 "GND" H 2200 5250 50  0000 C CNN
 F 2 "" H 2200 5400 50  0000 C CNN
@@
 NoConn ~ 8600 2400
 $Comp
-L GND #PWR03
+L GND #PWR2
 U 1 1 58F8B2B9
 P 8100 3000
-F 0 "#PWR03" H 8100 2750 50  0001 C CNN
+F 0 "#PWR2" H 8100 2750 50  0001 C CNN
 F 1 "GND" H 8100 2850 50  0000 C CNN
 F 2 "" H 8100 3000 50  0000 C CNN
@@
 LOAD+
 $Comp
-L GND #PWR04
+L GND #PWR3
 U 1 1 58F8D990
 P 9900 3000
-F 0 "#PWR04" H 9900 2750 50  0001 C CNN
+F 0 "#PWR3" H 9900 2750 50  0001 C CNN
 F 1 "GND" H 9900 2850 50  0000 C CNN
 F 2 "" H 9900 3000 50  0000 C CNN
@@
 NoConn ~ 9800 2800
 $Comp
-L GND #PWR05
+L GND #PWR4
 U 1 1 58F8DC25
 P 10400 3700
-F 0 "#PWR05" H 10400 3450 50  0001 C CNN
+F 0 "#PWR4" H 10400 3450 50  0001 C CNN
 F 1 "GND" H 10400 3550 50  0000 C CNN
 F 2 "" H 10400 3700 50  0000 C CNN
@@
 	5200 1600 5200 1500
 Wire Wire Line
-	5200 1500 4800 1500
+	5200 1500 4900 1500
+Wire Wire Line
+	4900 1500 4500 1500
 Wire Wire Line
 	2200 5400 2200 5300
@@
 	4500 1900 4600 1900
 Wire Wire Line
-	4600 1900 5000 1900
+	4600 1900 4900 1900
+Wire Wire Line
+	4900 1900 5000 1900
 Wire Wire Line
 	4500 1900 4500 1600
@@
 Text Notes 3200 4700 0    50   ~ 0
 Only populate 2 resistors\nfor 50A nominal!
-Text Notes 1400 1500 0    50   ~ 0
-Maximum voltage: 36 V\n(--> only suitable for up to 8 LiFePO4 cells)\nMaximum current: 50 A continuous, 100 A peak
+Text Notes 1200 1300 0    50   ~ 0
+Maximum voltage: 24 V\n(--> only suitable for up to 5 Li-Ion / Li Polymer cells)\nMaximum current: 50 A continuous, 100 A peak
 Text Notes 8600 1600 0    50   ~ 0
 Max. C_iss of CSD18540Q5B = 4.23 nF\n\nNecessary CP capacity acc. datasheet:\n4 x 4.23 nF x 470/20 = 0.4 uF
+$Comp
+L R R17
+U 1 1 59EC9161
+P 4900 1700
+F 0 "R17" V 4825 1700 50  0000 C CNN
+F 1 "1M" V 4975 1700 50  0000 C CNN
+F 2 "LibreSolar:R_0603_1608" V 4725 1600 50  0001 C CNN
+F 3 "" H 4900 1700 50  0000 C CNN
+F 4 "Yageo" H 100 -900 60  0001 C CNN "Manufacturer"
+F 5 "RC0603FR-071ML" H 100 -900 60  0001 C CNN "PartNumber"
+	1    4900 1700
+	1    0    0    1
+$EndComp
+Wire Wire Line
+	4900 1800 4900 1900
+Connection ~ 4900 1900
+Wire Wire Line
+	4900 1600 4900 1500
+Connection ~ 4900 1500
 $EndSCHEMATC
