File: power-pcb/Switch-N-Sense.sch (KiCad schematic (older format))
At the start: 41 parts, among them P1 CONN_01X01, P2 CONN_01X01, P3 CONN_01X01, P4 CONN_01X01, P5 CONN_01X01, P6 Conn_Switch-N-Sense, Q1 BSC010N04LS, Q2 BSC010N04LS, Q3 BSC010N04LS, Q4 BSC010N04LS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

Commit message: Small changes in power PCB
Changed lines of the file:
@@
 $EndComp
 $Comp
-L GND #PWR1
+L GND #PWR01
 U 1 1 58F8A6D0
 P 7900 3000
-F 0 "#PWR1" H 7900 2750 50  0001 C CNN
+F 0 "#PWR01" H 7900 2750 50  0001 C CNN
 F 1 "GND" H 7900 2850 50  0000 C CNN
 F 2 "" H 7900 3000 50  0000 C CNN
@@
 $EndComp
 $Comp
-L GND #PWR5
+L GND #PWR02
 U 1 1 58F8A862
 P 2200 5400
-F 0 "#PWR5" H 2200 5150 50  0001 C CNN
+F 0 "#PWR02" H 2200 5150 50  0001 C CNN
 F 1 "GND" H 2200 5250 50  0000 C CNN
 F 2 "" H 2200 5400 50  0000 C CNN
@@
 NoConn ~ 8600 2400
 $Comp
-L GND #PWR2
+L GND #PWR03
 U 1 1 58F8B2B9
 P 8100 3000
-F 0 "#PWR2" H 8100 2750 50  0001 C CNN
+F 0 "#PWR03" H 8100 2750 50  0001 C CNN
 F 1 "GND" H 8100 2850 50  0000 C CNN
 F 2 "" H 8100 3000 50  0000 C CNN
@@
 LOAD+
 $Comp
-L GND #PWR3
+L GND #PWR04
 U 1 1 58F8D990
 P 9900 3000
-F 0 "#PWR3" H 9900 2750 50  0001 C CNN
+F 0 "#PWR04" H 9900 2750 50  0001 C CNN
 F 1 "GND" H 9900 2850 50  0000 C CNN
 F 2 "" H 9900 3000 50  0000 C CNN
@@
 NoConn ~ 9800 2800
 $Comp
-L GND #PWR4
+L GND #PWR05
 U 1 1 58F8DC25
 P 10400 3700
-F 0 "#PWR4" H 10400 3450 50  0001 C CNN
+F 0 "#PWR05" H 10400 3450 50  0001 C CNN
 F 1 "GND" H 10400 3550 50  0000 C CNN
 F 2 "" H 10400 3700 50  0000 C CNN
@@
 BAT-
 Wire Wire Line
-	1800 2800 2000 2800
-Wire Wire Line
-	2000 2800 2300 2800
-Wire Wire Line
-	2300 2800 2800 2800
-Wire Wire Line
-	3200 2800 3400 2800
-Wire Wire Line
-	3400 2800 3500 2800
-Wire Wire Line
-	3500 2800 3900 2800
-Wire Wire Line
-	3900 2800 4100 2800
-Wire Wire Line
-	3200 3500 3500 3500
-Wire Wire Line
-	3500 3500 4100 3500
+	1800 2800 2800 2800
+Wire Wire Line
+	3200 2800 4100 2800
+Wire Wire Line
+	3200 3500 4100 3500
 Connection ~ 3900 2800
 Wire Wire Line
@@
 Connection ~ 2300 2800
 Wire Wire Line
-	4500 2800 5000 2800
-Wire Wire Line
-	5000 2800 5400 2800
-Wire Wire Line
-	5400 2800 5600 2800
-Wire Wire Line
-	5600 2800 6000 2800
-Wire Wire Line
-	6000 2800 6300 2800
+	4500 2800 6300 2800
 Wire Wire Line
 	5000 3500 4500 3500
 Connection ~ 5000 2800
 Wire Wire Line
-	2300 2400 2700 2400
-Wire Wire Line
-	2700 2400 3000 2400
+	2300 2400 3000 2400
 Wire Wire Line
 	3000 2400 3000 2500
@@
 	2700 2400 2700 3100
 Wire Wire Line
-	2600 3100 2700 3100
-Wire Wire Line
-	2700 3100 3000 3100
+	2600 3100 3000 3100
 Wire Wire Line
 	3000 3100 3000 3200
@@
 	4300 2500 4300 2400
 Wire Wire Line
-	5000 2800 5000 3100
-Wire Wire Line
-	5000 3100 5000 3500
-Wire Wire Line
-	5000 3500 5000 3900
+	5000 2800 5000 3900
 Wire Wire Line
 	4600 2400 4600 3100
 Wire Wire Line
-	4300 3100 4600 3100
-Wire Wire Line
-	4600 3100 4700 3100
+	4300 3100 4700 3100
 Wire Wire Line
 	4300 3100 4300 3200
 Wire Wire Line
-	2300 2800 2300 3100
-Wire Wire Line
-	2300 3100 2300 3500
-Wire Wire Line
-	2300 3500 2300 3900
+	2300 2800 2300 3900
 Wire Wire Line
 	2400 3100 2300 3100
@@
 Connection ~ 5000 3100
 Wire Wire Line
-	4300 2400 4600 2400
-Wire Wire Line
-	4600 2400 5000 2400
+	4300 2400 5000 2400
 Wire Wire Line
 	5600 1900 5600 2800
@@
 	3600 4900 3800 4900
 Wire Wire Line
-	3800 4900 3800 5200
-Wire Wire Line
-	3800 5200 3800 5300
-Wire Wire Line
-	3800 5300 3800 5500
-Wire Wire Line
-	3800 5500 3800 5800
+	3800 4900 3800 5800
 Wire Wire Line
 	3800 5800 3600 5800
@@
 Connection ~ 3800 5200
 Wire Wire Line
-	3800 5300 5400 5300
-Wire Wire Line
-	5400 5300 6000 5300
-Wire Wire Line
-	6000 5300 6300 5300
+	3800 5300 6300 5300
 Connection ~ 3800 5300
 Wire Wire Line
 	3400 4900 3200 4900
 Wire Wire Line
-	3200 4900 3200 5200
-Wire Wire Line
-	3200 5200 3200 5300
-Wire Wire Line
-	3200 5300 3200 5500
-Wire Wire Line
-	3200 5500 3200 5800
+	3200 4900 3200 5800
 Wire Wire Line
 	3200 5800 3400 5800
@@
 Connection ~ 3200 5500
 Wire Wire Line
-	1800 5300 2000 5300
-Wire Wire Line
-	2000 5300 2200 5300
-Wire Wire Line
-	2200 5300 3200 5300
+	1800 5300 3200 5300
 Connection ~ 3200 5300
 Wire Wire Line
@@
 Connection ~ 2700 2400
 Wire Wire Line
-	5200 1600 5200 1500
-Wire Wire Line
-	5200 1500 4900 1500
-Wire Wire Line
-	4900 1500 4500 1500
+	5200 1500 5200 1600
+Wire Wire Line
+	4500 1500 5200 1500
 Wire Wire Line
 	2200 5400 2200 5300
@@
 	8600 2600 8100 2600
 Wire Wire Line
-	7900 2300 8100 2300
-Wire Wire Line
-	8100 2300 8600 2300
-Wire Wire Line
-	7900 2200 7900 2300
-Wire Wire Line
-	7900 2300 7900 2500
+	7900 2300 8600 2300
+Wire Wire Line
+	7900 2200 7900 2500
 Connection ~ 7900 2300
 Wire Wire Line
@@
 	8600 2900 8300 2900
 Wire Wire Line
-	8100 2600 8100 2800
-Wire Wire Line
-	8100 2800 8100 3000
+	8100 2600 8100 3000
 Connection ~ 8100 2800
 Wire Wire Line
@@
 	10400 3000 10400 2700
 Wire Wire Line
-	10400 3200 10400 3300
-Wire Wire Line
-	10400 3300 10400 3400
+	10400 3200 10400 3400
 Wire Wire Line
 	10400 3300 10100 3300
@@
 	5600 1900 5400 1900
 Wire Wire Line
-	4300 1900 4500 1900
-Wire Wire Line
-	4500 1900 4600 1900
-Wire Wire Line
-	4600 1900 4900 1900
-Wire Wire Line
-	4900 1900 5000 1900
+	4300 1900 5000 1900
 Wire Wire Line
 	4500 1900 4500 1600
@@
 	4100 1600 3900 1600
 Wire Wire Line
-	3900 1600 3900 1900
-Wire Wire Line
-	3900 1900 3900 2200
-Wire Wire Line
-	3900 2200 3900 2800
+	3900 1600 3900 2800
 Wire Wire Line
 	3900 1900 4100 1900
