File: power-pcb/Switch-N-Sense.sch (KiCad schematic (older format))
At the start: 40 parts, among them P1 CONN_01X01, P2 CONN_01X01, P3 CONN_01X01, P4 CONN_01X01, P5 CONN_01X01, P6 Conn_Switch-N-Sense, Q1 CSD18540Q5B, Q2 CSD18540Q5B, Q3 CSD18540Q5B, Q4 CSD18540Q5B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

Commit message: Issues #1, #2 and #4 fixed
Parts:
- R7: PartNumber RC2010JK-0733RL -> RC2010JK-07330RL
Changed lines of the file:
@@
 EESchema Schematic File Version 2
+LIBS:Switch-N-Sense-rescue
 LIBS:IEC-60617
 LIBS:LibreSolar
@@
 F 3 "" H 4200 2200 50  0000 C CNN
 F 4 "Yageo" H 4200 2200 60  0001 C CNN "Manufacturer"
-F 5 "RC2010JK-0733RL" H 4200 2200 60  0001 C CNN "PartNumber"
+F 5 "RC2010JK-07330RL" H 4200 2200 60  0001 C CNN "PartNumber"
 	1    4200 2200
 	0    1    1    0
@@
 BAT-
 Wire Wire Line
-	1800 2800 2800 2800
-Wire Wire Line
-	3200 2800 4100 2800
-Wire Wire Line
-	3200 3500 4100 3500
+	1800 2800 2000 2800
+Wire Wire Line
+	2000 2800 2300 2800
+Wire Wire Line
+	2300 2800 2800 2800
+Wire Wire Line
+	3200 2800 3400 2800
+Wire Wire Line
+	3400 2800 3500 2800
+Wire Wire Line
+	3500 2800 3900 2800
+Wire Wire Line
+	3900 2800 4100 2800
+Wire Wire Line
+	3200 3500 3500 3500
+Wire Wire Line
+	3500 3500 4100 3500
 Connection ~ 3900 2800
 Wire Wire Line
@@
 Connection ~ 2300 2800
 Wire Wire Line
-	4500 2800 6300 2800
+	4500 2800 5000 2800
+Wire Wire Line
+	5000 2800 5400 2800
+Wire Wire Line
+	5400 2800 5600 2800
+Wire Wire Line
+	5600 2800 6000 2800
+Wire Wire Line
+	6000 2800 6300 2800
 Wire Wire Line
 	5000 3500 4500 3500
 Connection ~ 5000 2800
 Wire Wire Line
-	2300 2400 3000 2400
+	2300 2400 2700 2400
+Wire Wire Line
+	2700 2400 3000 2400
 Wire Wire Line
 	3000 2400 3000 2500
@@
 	2700 2400 2700 3100
 Wire Wire Line
-	2600 3100 3000 3100
+	2600 3100 2700 3100
+Wire Wire Line
+	2700 3100 3000 3100
 Wire Wire Line
 	3000 3100 3000 3200
@@
 	4300 2500 4300 2400
 Wire Wire Line
-	5000 2800 5000 3900
+	5000 2800 5000 3100
+Wire Wire Line
+	5000 3100 5000 3500
+Wire Wire Line
+	5000 3500 5000 3900
 Wire Wire Line
 	4600 2400 4600 3100
 Wire Wire Line
-	4300 3100 4700 3100
+	4300 3100 4600 3100
+Wire Wire Line
+	4600 3100 4700 3100
 Wire Wire Line
 	4300 3100 4300 3200
 Wire Wire Line
-	2300 2800 2300 3900
+	2300 2800 2300 3100
+Wire Wire Line
+	2300 3100 2300 3500
+Wire Wire Line
+	2300 3500 2300 3900
 Wire Wire Line
 	2400 3100 2300 3100
@@
 Connection ~ 5000 3100
 Wire Wire Line
-	4300 2400 5000 2400
+	4300 2400 4600 2400
+Wire Wire Line
+	4600 2400 5000 2400
 Wire Wire Line
 	5600 1900 5600 2800
@@
 	3600 4900 3800 4900
 Wire Wire Line
-	3800 4900 3800 5800
+	3800 4900 3800 5200
+Wire Wire Line
+	3800 5200 3800 5300
+Wire Wire Line
+	3800 5300 3800 5500
+Wire Wire Line
+	3800 5500 3800 5800
 Wire Wire Line
 	3800 5800 3600 5800
@@
 Connection ~ 3800 5200
 Wire Wire Line
-	3800 5300 6300 5300
+	3800 5300 5400 5300
+Wire Wire Line
+	5400 5300 6000 5300
+Wire Wire Line
+	6000 5300 6300 5300
 Connection ~ 3800 5300
 Wire Wire Line
 	3400 4900 3200 4900
 Wire Wire Line
-	3200 4900 3200 5800
+	3200 4900 3200 5200
+Wire Wire Line
+	3200 5200 3200 5300
+Wire Wire Line
+	3200 5300 3200 5500
+Wire Wire Line
+	3200 5500 3200 5800
 Wire Wire Line
 	3200 5800 3400 5800
@@
 Connection ~ 3200 5500
 Wire Wire Line
-	1800 5300 3200 5300
+	1800 5300 2000 5300
+Wire Wire Line
+	2000 5300 2200 5300
+Wire Wire Line
+	2200 5300 3200 5300
 Connection ~ 3200 5300
 Wire Wire Line
@@
 	8600 2600 8100 2600
 Wire Wire Line
-	7900 2300 8600 2300
-Wire Wire Line
-	7900 2200 7900 2500
+	7900 2300 8100 2300
+Wire Wire Line
+	8100 2300 8600 2300
+Wire Wire Line
+	7900 2200 7900 2300
+Wire Wire Line
+	7900 2300 7900 2500
 Connection ~ 7900 2300
 Wire Wire Line
@@
 	8600 2900 8300 2900
 Wire Wire Line
-	8100 2600 8100 3000
+	8100 2600 8100 2800
+Wire Wire Line
+	8100 2800 8100 3000
 Connection ~ 8100 2800
 Wire Wire Line
@@
 	10400 3000 10400 2700
 Wire Wire Line
-	10400 3200 10400 3400
+	10400 3200 10400 3300
+Wire Wire Line
+	10400 3300 10400 3400
 Wire Wire Line
 	10400 3300 10100 3300
@@
 	5600 1900 5400 1900
 Wire Wire Line
-	4300 1900 5000 1900
+	4300 1900 4500 1900
+Wire Wire Line
+	4500 1900 4600 1900
+Wire Wire Line
+	4600 1900 5000 1900
 Wire Wire Line
 	4500 1900 4500 1600
@@
 	4100 1600 3900 1600
 Wire Wire Line
-	3900 1600 3900 2800
+	3900 1600 3900 1900
+Wire Wire Line
+	3900 1900 3900 2200
+Wire Wire Line
+	3900 2200 3900 2800
 Wire Wire Line
 	3900 1900 4100 1900

Commit message: Update to KiCAD 5 and minor changes in part selection
Parts:
- removed P1: CONN_01X01, LibreSolar:Wuerth_WP-THRBU, symbol CONN_01X01
- removed R3, R4: 2m, LibreSolar:R_Bourns_CRE2512, symbol R
- C1: footprint LibreSolar:C_0603_1608 -> LibreSolar:C_0805_2012; symbol C -> Project:C; Manufacturer Murata -> Yageo; PartNumber GRM188R61H105KAALD -> CC0603KRX7R8BB105
- C2, C5: symbol C -> Project:C; Manufacturer Murata -> Yageo; PartNumber GRM188R71H103KA01D -> CC0603KRX7R9BB103
- C3, C4, C6, C7: symbol C -> Project:C; Manufacturer Murata -> Yageo; PartNumber GRM188R71H104KA93D -> CC0603KRX7R9BB104
- D1, D2: value SMCJ36A -> SMCJ24A; symbol D_Schottky -> Project:D_Schottky; PartNumber SMCJ36A -> SMCJ24A
- LOGO1: symbol LIBRE_SOLAR -> Project:LibreSolar_Logo
- LOGO2: footprint Symbols:OSHW-Logo_5.7x6mm_SilkScreen -> Symbol:OSHW-Logo_5.7x6mm_SilkScreen; symbol OPEN_HARDWARE_1 -> Project:Logo_Open_Hardware_Small
- P2, P3, P4, P5: symbol CONN_01X01 -> Project:Conn_01x01; Manufacturer Würth -> Wuerth
- P6: symbol Conn_Switch-N-Sense_Inverted -> Project:Conn_Switch-N-Sense_Inverted; Manufacturer Würth -> Wuerth
- Q1, Q2, Q3, Q4: value CSD18540Q5B -> BSC014N04LS; symbol Q_NMOS -> LibreSolar:Q_NMOS; Manufacturer Texas Instruments -> Infineon; PartNumber CSD18540Q5B -> BSC014N04LS
- Q5: value ZXMP10A13F -> ZXMP6A13F; symbol Q_PMOS_GDS -> Project:Q_PMOS_GSD; PartNumber ZXMP10A13FTA -> ZXMP6A13FTA; Remarks (none) -> -60V
- R1, R10, R11, R12, R13, R14, R15, R16, R2, R7, R8, R9: symbol R -> Project:R
- R5, R6: symbol R -> Project:R; PartNumber RC2010JK-0733RL -> RC2010JK-07330RL
- RT1: symbol Thermistor_NTC -> Project:R_NTC
- U1: footprint Housings_SSOP:TSSOP-16_4.4x5mm_Pitch0.65mm -> Package_SO:TSSOP-16_4.4x5mm_P0.65mm; symbol BQ76200 -> Project:BQ76200
Connections:
- wire segments 141 -> 131
Other:
- note added: "BSC014N04LS (1.4 mOhm) or \nBSC010N04LS (1 mOhm)"
- note added: "Maximum voltage: 24 V (5s BMS)\nMaximum current: 50 A continuous, 100 A peak"
- note removed: "Maximum voltage: 36 V\n(--> only suitable for up to 8 LiFePO4 cells)\nMaximum current: 50 A continuous, 100 A peak"
- moved on the sheet: C3, C4, R1, R2
