File: control-pcb/analog_frontend.sch (KiCad schematic (older format))
At the start: 16 parts, among them P6 CONN_01X02, P7 CONN_01X02

Commit message: Update to KiCAD 5 and minor changes in part selection
Parts:
- C37, C38, C39, C40: symbol C -> Project:C; Manufacturer Murata -> Yageo; PartNumber GRM188R71H104KA93D -> CC0603KRX7R9BB104
- D18, D19, D20, D21: symbol D_Zener -> Project:D_Zener
- P6, P7: symbol CONN_01X02 -> Project:Conn_01x02
- R43, R44, R45, R46, R47, R48: symbol R -> Project:R
Connections:
- wire segments 36 -> 48
Changed lines of the file:
@@
-EESchema Schematic File Version 2
-LIBS:IEC-60617
-LIBS:LibreSolar
-LIBS:power
-LIBS:device
-LIBS:conn
-LIBS:logo
+EESchema Schematic File Version 4
 LIBS:BMS-5s-cache
 EELAYER 26 0
@@
 $EndDescr
 $Comp
-L GND #PWR078
+L power:GND #PWR078
 U 1 1 58A6D4FE
 P 2300 6200
@@
 $EndComp
 $Comp
-L GND #PWR079
+L power:GND #PWR079
 U 1 1 58A6DA9F
 P 2700 6200
@@
 $EndComp
 $Comp
-L C C39
+L Project:C C39
 U 1 1 58A7377B
 P 2300 5900
@@
 F 2 "LibreSolar:C_0603_1608" H 2300 5700 50  0001 C CNN
 F 3 "" H 2325 5975 50  0000 C CNN
-F 4 "Murata" H -6500 50  50  0001 C CNN "Manufacturer"
-F 5 "GRM188R71H104KA93D" H -6500 50  50  0001 C CNN "PartNumber"
+F 4 "Yageo" H -6500 50  50  0001 C CNN "Manufacturer"
+F 5 "CC0603KRX7R9BB104" H -6500 50  50  0001 C CNN "PartNumber"
 	1    2300 5900
 	1    0    0    -1
 $EndComp
 $Comp
-L +3.3V #PWR080
+L power:+3.3V #PWR080
 U 1 1 58A73CA0
 P 2700 5100
@@
 $EndComp
 $Comp
-L R R47
+L Project:R R47
 U 1 1 58A7452B
 P 2700 5300
@@
 $EndComp
 $Comp
-L GND #PWR081
+L power:GND #PWR081
 U 1 1 58C07122
 P 4800 6200
@@
 $EndComp
 $Comp
-L C C40
+L Project:C C40
 U 1 1 58CBE39F
 P 4400 5950
@@
 F 2 "LibreSolar:C_0603_1608" H 4400 5750 50  0001 C CNN
 F 3 "" H 4425 6025 50  0000 C CNN
-F 4 "Murata" H -5650 100 50  0001 C CNN "Manufacturer"
-F 5 "GRM188R71H104KA93D" H -5650 100 50  0001 C CNN "PartNumber"
+F 4 "Yageo" H -5650 100 50  0001 C CNN "Manufacturer"
+F 5 "CC0603KRX7R9BB104" H -5650 100 50  0001 C CNN "PartNumber"
 	1    4400 5950
 	1    0    0    -1
 $EndComp
 $Comp
-L GND #PWR082
+L power:GND #PWR082
 U 1 1 58CBE489
 P 4400 6200
@@
 $EndComp
 $Comp
-L R R48
+L Project:R R48
 U 1 1 58CBE7D6
 P 4800 5300
@@
 $EndComp
 $Comp
-L +3.3V #PWR083
+L power:+3.3V #PWR083
 U 1 1 58CBE8D7
 P 4800 5100
@@
 	2300 5800 2300 5600
 Wire Wire Line
-	1900 5600 2800 5600
+	1900 5600 2300 5600
 Wire Wire Line
 	4800 5100 4800 5200
 Wire Wire Line
-	4000 5600 4900 5600
+	4000 5600 4400 5600
 Wire Wire Line
 	4400 6050 4400 6200
@@
 Temperature (ext./int.)
 $Comp
-L R R45
+L Project:R R45
 U 1 1 58E84BA2
 P 2600 2600
@@
 F 2 "LibreSolar:R_0603_1608" V 2425 2500 50  0001 C CNN
 F 3 "" H 2600 2600 50  0000 C CNN
-F 4 "RC0603FR-0710KL" H 2600 2600 60  0001 C CNN "PartNumber"
-F 5 "Yageo" H 0   0   60  0001 C CNN "Manufacturer"
+F 4 "Yageo" H 0   0   60  0001 C CNN "Manufacturer"
+F 5 "RC0603FR-0710KL" H 2600 2600 60  0001 C CNN "PartNumber"
 	1    2600 2600
 	1    0    0    -1
 $EndComp
 $Comp
-L R R43
+L Project:R R43
 U 1 1 58E84BA9
 P 2600 2000
@@
 $EndComp
 $Comp
-L R R46
+L Project:R R46
 U 1 1 58E84BB0
 P 4200 2600
@@
 F 2 "LibreSolar:R_0603_1608" V 4025 2500 50  0001 C CNN
 F 3 "" H 4200 2600 50  0000 C CNN
-F 4 "RC0603FR-0710KL" H 4200 2600 60  0001 C CNN "PartNumber"
-F 5 "Yageo" H 300 0   60  0001 C CNN "Manufacturer"
+F 4 "Yageo" H 300 0   60  0001 C CNN "Manufacturer"
+F 5 "RC0603FR-0710KL" H 4200 2600 60  0001 C CNN "PartNumber"
 	1    4200 2600
 	1    0    0    -1
 $EndComp
 $Comp
-L R R44
+L Project:R R44
 U 1 1 58E84BB7
 P 4200 2000
@@
 $EndComp
 $Comp
-L C C37
+L Project:C C37
 U 1 1 58E84BBE
 P 2900 2600
@@
 F 2 "LibreSolar:C_0603_1608" H 2900 2400 50  0001 C CNN
 F 3 "" H 2925 2675 50  0000 C CNN
-F 4 "Murata" H 0   0   60  0001 C CNN "Manufacturer"
-F 5 "GRM188R71H104KA93D" H 0   0   60  0001 C CNN "PartNumber"
+F 4 "Yageo" H 0   0   60  0001 C CNN "Manufacturer"
+F 5 "CC0603KRX7R9BB104" H 0   0   60  0001 C CNN "PartNumber"
 	1    2900 2600
 	1    0    0    -1
 $EndComp
 $Comp
-L C C38
+L Project:C C38
 U 1 1 58E84BC5
 P 4500 2600
@@
 F 2 "LibreSolar:C_0603_1608" H 4500 2400 50  0001 C CNN
 F 3 "" H 4525 2675 50  0000 C CNN
-F 4 "Murata" H 0   0   60  0001 C CNN "Manufacturer"
-F 5 "GRM188R71H104KA93D" H 0   0   60  0001 C CNN "PartNumber"
+F 4 "Yageo" H 0   0   60  0001 C CNN "Manufacturer"
+F 5 "CC0603KRX7R9BB104" H 0   0   60  0001 C CNN "PartNumber"
 	1    4500 2600
 	1    0    0    -1
@@
 Battery and load voltage
 $Comp
-L GND #PWR084
+L power:GND #PWR084
 U 1 1 58E84BCD
 P 4500 2900
@@
 $EndComp
 $Comp
-L GND #PWR085
+L power:GND #PWR085
 U 1 1 58E84BD3
 P 4200 2900
@@
 $EndComp
 $Comp
-L GND #PWR086
+L power:GND #PWR086
 U 1 1 58E84BD9
 P 2900 2900
@@
 $EndComp
 $Comp
-L GND #PWR087
+L power:GND #PWR087
 U 1 1 58E84BDF
 P 2600 2900
@@
 Connection ~ 4200 2300
 Wire Wire Line
-	4200 2300 5000 2300
+	4200 2300 4500 2300
 Wire Wire Line
 	4500 2300 4500 2500
@@
 	4200 2700 4200 2900
 Wire Wire Line
-	4200 2100 4200 2500
+	4200 2100 4200 2300
 Connection ~ 2600 2300
 Wire Wire Line
-	2600 2300 3400 2300
+	2600 2300 2900 2300
 Wire Wire Line
 	2900 2300 2900 2500
@@
 	2600 2700 2600 2900
 Wire Wire Line
-	2600 2100 2600 2500
+	2600 2100 2600 2300
 Wire Wire Line
 	2600 1700 2600 1900
@@
 	4400 5850 4400 5600
 $Comp
-L CONN_01X02 P6
+L Project:Conn_01x02 P6
 U 1 1 5912D5A4
-P 3100 5950
-F 0 "P6" H 3100 6100 50  0000 C CNN
-F 1 "CONN_01X02" V 3200 5950 50  0000 C CNN
-F 2 "LibreSolar:Phoenix_Contact_MC_1,5_2-G-3,81" H 3100 5950 50  0001 C CNN
-F 3 "" H 3100 5950 50  0000 C CNN
-F 4 "Phoenix Contact" H 0   0   60  0001 C CNN "Manufacturer"
-F 5 "1803277" H 0   0   60  0001 C CNN "PartNumber"
-	1    3100 5950
-	1    0    0    -1
-$EndComp
-$Comp
-L CONN_01X02 P7
+P 3100 5900
+F 0 "P6" H 3100 6050 50  0000 C CNN
+F 1 "CONN_01X02" V 3200 5900 50  0000 C CNN
+F 2 "LibreSolar:Phoenix_Contact_MC_1,5_2-G-3,81" H 3100 5900 50  0001 C CNN
+F 3 "" H 3100 5900 50  0000 C CNN
+F 4 "Phoenix Contact" H 0   -50 60  0001 C CNN "Manufacturer"
+F 5 "1803277" H 0   -50 60  0001 C CNN "PartNumber"
+	1    3100 5900
+	1    0    0    -1
+$EndComp
+$Comp
+L Project:Conn_01x02 P7
 U 1 1 5912D60E
-P 5200 5950
-F 0 "P7" H 5200 6100 50  0000 C CNN
-F 1 "CONN_01X02" V 5300 5950 50  0000 C CNN
-F 2 "LibreSolar:Phoenix_Contact_MC_1,5_2-G-3,81" H 5200 5950 50  0001 C CNN
-F 3 "" H 5200 5950 50  0000 C CNN
-F 4 "Phoenix Contact" H 5200 5950 60  0001 C CNN "Manufacturer"
-F 5 "1803277" H 5200 5950 60  0001 C CNN "PartNumber"
-	1    5200 5950
+P 5200 5900
+F 0 "P7" H 5200 6050 50  0000 C CNN
+F 1 "CONN_01X02" V 5300 5900 50  0000 C CNN
+F 2 "LibreSolar:Phoenix_Contact_MC_1,5_2-G-3,81" H 5200 5900 50  0001 C CNN
+F 3 "" H 5200 5900 50  0000 C CNN
+F 4 "Phoenix Contact" H 5200 5900 60  0001 C CNN "Manufacturer"
+F 5 "1803277" H 5200 5900 60  0001 C CNN "PartNumber"
+	1    5200 5900
 	1    0    0    -1
 $EndComp
@@
 	2700 5900 2900 5900
 Wire Wire Line
-	2700 5400 2700 5900
+	2700 5400 2700 5600
 Wire Wire Line
 	4800 5900 5000 5900
 Wire Wire Line
-	4800 5400 4800 5900
+	4800 5400 4800 5600
 Wire Wire Line
 	5000 6000 4800 6000
@@
 	4800 6000 4800 6200
 $Comp
-L D_Zener D18
+L Project:D_Zener D18
 U 1 1 59166422
 P 1900 5900
@@
 	1900 5600 1900 5800
 $Comp
-L GND #PWR088
+L power:GND #PWR088
 U 1 1 591664BD
 P 1900 6200
@@
 $EndComp
 $Comp
-L D_Zener D19
+L Project:D_Zener D19
 U 1 1 59166596
 P 4000 5900
@@
 	4000 5600 4000 5800
 $Comp
-L GND #PWR089
+L power:GND #PWR089
 U 1 1 5916659E
 P 4000 6200
@@
 Maximum voltage: 5*4.2V = 21V\n
 $Comp
-L D_Zener D21
+L Project:D_Zener D21
 U 1 1 59221F12
 P 4800 2600
@@
 $EndComp
 $Comp
-L D_Zener D20
+L Project:D_Zener D20
 U 1 1 5922209E
 P 3200 2600
@@
 $EndComp
 $Comp
-L GND #PWR090
+L power:GND #PWR090
 U 1 1 5922226C
 P 4800 2900
@@
 $EndComp
 $Comp
-L GND #PWR091
+L power:GND #PWR091
 U 1 1 59222297
 P 3200 2900
@@
 Wire Wire Line
 	4800 2700 4800 2900
+Wire Wire Line
+	2700 5600 2800 5600
+Wire Wire Line
+	2700 5600 2700 5900
+Wire Wire Line
+	4800 5600 4900 5600
+Wire Wire Line
+	4800 5600 4800 5900
+Wire Wire Line
+	2900 2300 3200 2300
+Wire Wire Line
+	4500 2300 4800 2300
+Wire Wire Line
+	4200 2300 4200 2500
+Wire Wire Line
+	2600 2300 2600 2500
+Wire Wire Line
+	4400 5600 4800 5600
+Wire Wire Line
+	2300 5600 2700 5600
+Wire Wire Line
+	3200 2300 3400 2300
+Wire Wire Line
+	4800 2300 5000 2300
 $EndSCHEMATC
