File: control-pcb/interfaces.sch (KiCad schematic (older format))
At the start: 16 parts, among them J2 UEXT, P4 USB_Micro-B, U4 TJA1042T/3

Commit message: Update to KiCAD 5 and minor changes in part selection
Parts:
- C24, C25, C26: symbol C -> Project:C; Manufacturer Murata -> Yageo; PartNumber GRM188R71H104KA93D -> CC0603KRX7R9BB104
- D15: footprint TO_SOT_Packages_SMD:SOT-23-6 -> LibreSolar:SOT-23-6; symbol USBLC6-2SC6 -> LibreSolar:USBLC6-2SC6
- D16: symbol NUP2105L -> Project:NUP2105L
- J2: symbol UEXT -> LibreSolar:UEXT
- JP1: footprint Pin_Headers:Pin_Header_Angled_2x01_Pitch2.54mm -> Connector_PinHeader_2.54mm:PinHeader_2x01_P2.54mm_Horizontal; symbol Jumper_NC_Small -> Project:Jumper_NC_Small
- JP2, JP3: symbol RJ45_NS -> Project:RJ45_NS
- P4: symbol USB_OTG -> Project:USB_OTG
- R31, R32, R33, R34: symbol R -> Project:R
- RT1: symbol R_PTC -> LibreSolar:R_PTC
- U4: footprint Housings_SOIC:SOIC-8_3.9x4.9mm_Pitch1.27mm -> LibreSolar:SOIC-8_3.9x4.9mm_Pitch1.27mm; symbol TJA1042T/3 -> Project:TJA1042T-3; Supplier (none) -> Mouser
Connections:
- wire segments 76 -> 78
Changed lines of the file:
@@
-EESchema Schematic File Version 2
-LIBS:IEC-60617
-LIBS:LibreSolar
-LIBS:power
-LIBS:device
-LIBS:conn
-LIBS:logo
+EESchema Schematic File Version 4
 LIBS:BMS-5s-cache
 EELAYER 26 0
@@
 $EndDescr
 $Comp
-L +3.3V #PWR034
+L power:+3.3V #PWR034
 U 1 1 58BE341B
 P 6300 1900
@@
 $EndComp
 $Comp
-L +5V #PWR035
+L power:+5V #PWR035
 U 1 1 58BE3421
 P 6000 1900
@@
 $EndComp
 $Comp
-L GND #PWR036
+L power:GND #PWR036
 U 1 1 58BE3427
 P 6300 2300
@@
 $EndComp
 $Comp
-L GND #PWR037
+L power:GND #PWR037
 U 1 1 58BE342E
 P 6000 2300
@@
 $EndComp
 $Comp
-L GND #PWR038
+L power:GND #PWR038
 U 1 1 58BE3434
 P 10300 2300
@@
 $EndComp
 $Comp
-L C C25
+L Project:C C25
 U 1 1 58BE3440
 P 6300 2100
@@
 F 2 "LibreSolar:C_0603_1608" H 6300 2100 50  0001 C CNN
 F 3 "" H 6300 2100 50  0000 C CNN
-F 4 "Murata" H -500 350 50  0001 C CNN "Manufacturer"
-F 5 "GRM188R71H104KA93D" H -500 350 50  0001 C CNN "PartNumber"
+F 4 "Yageo" H -500 350 50  0001 C CNN "Manufacturer"
+F 5 "CC0603KRX7R9BB104" H -500 350 50  0001 C CNN "PartNumber"
 	1    6300 2100
 	1    0    0    -1
 $EndComp
 $Comp
-L C C24
+L Project:C C24
 U 1 1 58BE3447
 P 6000 2100
@@
 F 2 "LibreSolar:C_0603_1608" H 6000 2100 50  0001 C CNN
 F 3 "" H 6000 2100 50  0000 C CNN
-F 4 "Murata" H -400 350 50  0001 C CNN "Manufacturer"
-F 5 "GRM188R71H104KA93D" H -400 350 50  0001 C CNN "PartNumber"
+F 4 "Yageo" H -400 350 50  0001 C CNN "Manufacturer"
+F 5 "CC0603KRX7R9BB104" H -400 350 50  0001 C CNN "PartNumber"
 	1    6000 2100
 	1    0    0    -1
 $EndComp
 $Comp
-L R R32
+L Project:R R32
 U 1 1 58BE344E
 P 8900 2300
@@
 $EndComp
 $Comp
-L RJ45_NS JP2
+L Project:RJ45_NS JP2
 U 1 1 58BE345B
 P 7050 3650
@@
 $EndComp
 $Comp
-L TJA1042T/3 U4
+L Project:TJA1042T-3 U4
 U 1 1 58BE3467
 P 7700 2200
 F 0 "U4" H 7700 2650 50  0000 C CNN
 F 1 "TJA1042T/3" H 7700 1850 50  0000 C CNN
-F 2 "Housings_SOIC:SOIC-8_3.9x4.9mm_Pitch1.27mm" H 7700 1700 50  0001 C CIN
+F 2 "LibreSolar:SOIC-8_3.9x4.9mm_Pitch1.27mm" H 7700 1700 50  0001 C CIN
 F 3 "" H 7700 2200 50  0000 C CNN
 F 4 "NXP" H -250 450 50  0001 C CNN "Manufacturer"
 F 5 "TJA1042T/3/1J" H -250 450 50  0001 C CNN "PartNumber"
+F 6 "Mouser" H 7700 2200 60  0001 C CNN "Supplier"
 	1    7700 2200
 	1    0    0    -1
 $EndComp
 $Comp
-L Jumper_NC_Small JP1
+L Project:Jumper_NC_Small JP1
 U 1 1 58BE3476
 P 8900 2000
 F 0 "JP1" H 8900 2080 50  0000 C CNN
 F 1 "Jumper_NC_Small" H 8910 1940 50  0001 C CNN
-F 2 "Pin_Headers:Pin_Header_Angled_2x01_Pitch2.54mm" H 8900 2000 50  0001 C CNN
+F 2 "Connector_PinHeader_2.54mm:PinHeader_2x01_P2.54mm_Horizontal" H 8900 2000 50  0001 C CNN
 F 3 "" H 8900 2000 50  0001 C CNN
 	1    8900 2000
@@
 $EndComp
 $Comp
-L RJ45_NS JP3
+L Project:RJ45_NS JP3
 U 1 1 58BE348A
 P 8650 3650
@@
 $EndComp
 $Comp
-L GND #PWR039
+L power:GND #PWR039
 U 1 1 58BE3F4D
 P 2200 3000
@@
 $EndComp
 $Comp
-L +3.3V #PWR040
+L power:+3.3V #PWR040
 U 1 1 58BE3F53
 P 2000 5400
@@
 $EndComp
 $Comp
-L GND #PWR041
+L power:GND #PWR041
 U 1 1 58BE3F59
 P 3600 5600
@@
 $EndComp
 $Comp
-L +3.3V #PWR042
+L power:+3.3V #PWR042
 U 1 1 58BE3F5F
 P 5050 5300
@@
 $EndComp
 $Comp
-L +3.3V #PWR043
+L power:+3.3V #PWR043
 U 1 1 58BE3F65
 P 4700 5300
@@
 $EndComp
 $Comp
-L R R34
+L Project:R R34
 U 1 1 58BE3F9C
 P 5050 5500
@@
 $EndComp
 $Comp
-L R R33
+L Project:R R33
 U 1 1 58BE3FA3
 P 4700 5500
@@
 $EndComp
 $Comp
-L UEXT J2
+L LibreSolar:UEXT J2
 U 1 1 58BDEEA0
 P 2500 5700
@@
 $EndComp
 $Comp
-L +3.3V #PWR044
+L power:+3.3V #PWR044
 U 1 1 58BDF61E
 P 7200 1800
@@
 $EndComp
 $Comp
-L +5V #PWR045
+L power:+5V #PWR045
 U 1 1 58BDF65F
 P 8200 1800
@@
 $EndComp
 $Comp
-L GND #PWR046
+L power:GND #PWR046
 U 1 1 58BDF6B3
 P 8200 2500
@@
 $EndComp
 $Comp
-L NUP2105L D16
+L Project:NUP2105L D16
 U 1 1 58BE0956
 P 9900 2200
@@
 $EndComp
 $Comp
-L USBLC6-2SC6 D15
+L LibreSolar:USBLC6-2SC6 D15
 U 1 1 58BE3F7F
 P 3300 2500
 F 0 "D15" H 3050 2850 50  0000 C CNN
 F 1 "USBLC6-2SC6" H 3300 2150 50  0000 C CNN
-F 2 "TO_SOT_Packages_SMD:SOT-23-6" H 3950 2850 50  0001 C CNN
+F 2 "LibreSolar:SOT-23-6" H 3950 2850 50  0001 C CNN
 F 3 "" H 3050 2850 50  0001 C CNN
 F 4 "STMicroelectronics" H 150 450 50  0001 C CNN "Manufacturer"
@@
 $EndComp
 $Comp
-L GND #PWR047
+L power:GND #PWR047
 U 1 1 58C190E2
 P 3950 2500
@@
 $EndComp
 $Comp
-L USB_OTG P4
+L Project:USB_OTG P4
 U 1 1 58CC2DA5
 P 1800 2400
@@
 $EndComp
 $Comp
-L C C26
+L Project:C C26
 U 1 1 58CC2EC7
 P 2000 2900
@@
 F 2 "LibreSolar:C_0603_1608" H 2000 2900 50  0001 C CNN
 F 3 "" H 2000 2900 50  0000 C CNN
-F 4 "Murata" H -1100 -200 50  0001 C CNN "Manufacturer"
-F 5 "GRM188R71H104KA93D" H -1100 -200 50  0001 C CNN "PartNumber"
+F 4 "Yageo" H -1100 -200 50  0001 C CNN "Manufacturer"
+F 5 "CC0603KRX7R9BB104" H -1100 -200 50  0001 C CNN "PartNumber"
 	1    2000 2900
 	0    1    -1   0
 $EndComp
 $Comp
-L GND #PWR048
+L power:GND #PWR048
 U 1 1 58CC340B
 P 2400 3000
@@
 $EndComp
 $Comp
-L R R31
+L Project:R R31
 U 1 1 58CC345E
 P 2400 2700
@@
 	2100 2900 2200 2900
 Wire Wire Line
-	2200 2600 2200 3000
+	2200 2600 2200 2900
 Connection ~ 2200 2900
 Wire Wire Line
@@
 	2600 2700 2800 2700
 Wire Wire Line
-	2100 2200 2700 2200
+	2100 2200 2200 2200
 Wire Wire Line
 	2700 2200 2700 2500
@@
 	2700 2500 2800 2500
 $Comp
-L +5V #PWR049
+L power:+5V #PWR049
 U 1 1 59167780
 P 2900 1800
@@
 $EndComp
 $Comp
-L R_PTC RT1
+L LibreSolar:R_PTC RT1
 U 1 1 59167F4E
 P 2500 1900
@@
 Text Label 6200 3700 0    50   ~ 0
 RJ45_P5
+Wire Wire Line
+	2200 2900 2200 3000
+Wire Wire Line
+	2200 2200 2700 2200
 $EndSCHEMATC
