File: control-pcb/bq76920.sch (KiCad schematic (older format))
At the start: 64 parts, among them P3 ON/OFF, Q1 DMN2004K, Q2 BSS84, Q3 DMN2004K, Q4 2N7002, Q5 DMN2004K, Q6 DMN2004K, Q7 DMN2004K, SW1 SW_PUSH, U1 BQ76920

Commit message: Issues #1, #2 and #4 fixed
Parts:
- Q4: value 2N7002 -> BSS138; Manufacturer Nexperia -> Fairchild Semiconductor; PartNumber 2N7002,215 -> BSS138
- SW1: Alternative (none) -> TE FSMRA3JH
Changed lines of the file:
@@
 EESchema Schematic File Version 2
-LIBS:BMS-5s-rescue
 LIBS:IEC-60617
 LIBS:LibreSolar
@@
 P 8900 2500
 F 0 "Q4" H 9200 2550 50  0000 R CNN
-F 1 "2N7002" H 9400 2450 50  0000 R CNN
+F 1 "BSS138" H 9400 2450 50  0000 R CNN
 F 2 "LibreSolar:SOT-23" H 9100 2600 50  0001 C CNN
 F 3 "" H 8900 2500 50  0000 C CNN
-F 4 "Nexperia" H 8900 2500 60  0001 C CNN "Manufacturer"
-F 5 "2N7002,215" H 8900 2500 60  0001 C CNN "PartNumber"
+F 4 "Fairchild Semiconductor" H 8900 2500 60  0001 C CNN "Manufacturer"
+F 5 "BSS138" H 8900 2500 60  0001 C CNN "PartNumber"
 	1    8900 2500
 	1    0    0    -1
@@
 F 4 "Würth" H 9100 4150 60  0001 C CNN "Manufacturer"
 F 5 "431256083716" H 9100 4150 60  0001 C CNN "PartNumber"
+F 6 "TE FSMRA3JH" H 9100 4150 60  0001 C CNN "Alternative"
 	1    9100 4150
 	0    1    1    0

Commit message: Update to KiCAD 5 and minor changes in part selection
Parts:
- C1, C11, C12, C13, C14, C2, C3, C4, C5, C6: symbol C -> Project:C; Manufacturer Murata -> Yageo; PartNumber GRM188R71H104KA93D -> CC0603KRX7R9BB104
- C10, C8: symbol C -> Project:C
- C7, C9: footprint LibreSolar:C_0603_1608 -> LibreSolar:C_0805_2012; symbol C -> Project:C; Manufacturer Murata -> Yageo; PartNumber GRM188R61H105KAALD -> CC0805KKX7R9BB105; Remarks X5R -> (none)
- D1, D10, D11, D12, D2, D3, D4, D5, D7, D9: symbol D_Zener -> Project:D_Zener
- D6, D8: symbol D -> Project:D
- P3: symbol CONN_01X02 -> Project:Conn_01x02
- Q1, Q3, Q4, Q5, Q6, Q7: symbol Q_NMOS_GSD -> Project:Q_NMOS_GSD
- Q2: symbol Q_PMOS_GSD -> Project:Q_PMOS_GSD
- R1, R10, R11, R12, R13, R14, R15, R16, R17, R18, R19, R2, R20, R21, R22, R23, R24, R25, R26, R3, R4, R49, R5, R50, R6, R7, R8, R9: symbol R -> Project:R
- SW1: symbol SW_PUSH -> Project:SW_PUSH
- U1: footprint Housings_SSOP:TSSOP-20_4.4x6.5mm_Pitch0.65mm -> Package_SO:TSSOP-20_4.4x6.5mm_P0.65mm; symbol BQ76920 -> Project:BQ76920
Connections:
- wire segments 163 -> 227

Commit message: Diode part number corrected, closing issue #9
Parts:
- D6, D8: value 1N4148W-7-F -> 1N4148WS-7-F; PartNumber 1N4148W-7-F -> 1N4148WS-7-F
Changed lines of the file:
@@
 P 6800 1500
 F 0 "D6" H 6800 1600 50  0000 C CNN
-F 1 "1N4148W-7-F" H 6800 1400 50  0000 C CNN
+F 1 "1N4148WS-7-F" H 6800 1400 50  0000 C CNN
 F 2 "LibreSolar:D_SOD-323" V 6800 1500 50  0001 C CNN
 F 3 "" V 6800 1500 50  0000 C CNN
 F 4 "Diodes Inc." H 0   0   60  0001 C CNN "Manufacturer"
-F 5 "1N4148W-7-F" H 0   0   60  0001 C CNN "PartNumber"
+F 5 "1N4148WS-7-F" H 0   0   60  0001 C CNN "PartNumber"
 	1    6800 1500
 	-1   0    0    -1
@@
 P 9700 4600
 F 0 "D8" H 9700 4700 50  0000 C CNN
-F 1 "1N4148W-7-F" H 9700 4500 50  0000 C CNN
+F 1 "1N4148WS-7-F" H 9700 4500 50  0000 C CNN
 F 2 "LibreSolar:D_SOD-323" V 9700 4600 50  0001 C CNN
 F 3 "" V 9700 4600 50  0000 C CNN
 F 4 "Diodes Inc." H 0   0   60  0001 C CNN "Manufacturer"
-F 5 "1N4148W-7-F" H 0   0   60  0001 C CNN "PartNumber"
+F 5 "1N4148WS-7-F" H 0   0   60  0001 C CNN "PartNumber"
 	1    9700 4600
 	-1   0    0    1
