File: control-pcb/power_supply.sch (KiCad schematic (older format))
At the start: 19 parts, among them U2 MCP16331-CH, U3 AP2210-3.3

Commit message: Update to KiCAD 5 and minor changes in part selection
Parts:
- C15, C18: symbol C -> Project:C; Manufacturer Murata -> Yageo; PartNumber GRM188R71H104KA93D -> CC0603KRX7R9BB104
- C16, C21: footprint LibreSolar:C_0603_1608 -> LibreSolar:C_0805_2012; symbol C -> Project:C; Manufacturer Murata -> Yageo; PartNumber GRM188R61H105KAALD -> CC0805KKX7R9BB105; Remarks X5R -> (none)
- C17, C19, C20, C22: symbol C -> Project:C
- C23: symbol C -> Project:C; Manufacturer Murata -> Yageo; PartNumber GRM1885C2A101JA01D -> CC0603JRNPO9BN101
- D13: symbol D -> Project:D
- D14: footprint Diodes_SMD:D_PowerDI-123 -> Diode_SMD:D_PowerDI-123; symbol D_Schottky -> Project:D_Schottky
- L1: footprint Inductors_SMD:L_0805 -> Inductor_SMD:L_0805_2012Metric; symbol L -> Project:L
- L2: symbol L -> Project:L
- R27, R28: symbol R -> Project:R
- TP1, TP2: symbol TEST -> Connector:Test_Point
- U2: footprint TO_SOT_Packages_SMD:SOT-23-6 -> LibreSolar:SOT-23-6; symbol MCP16331-CH -> Project:MCP16331-CH
- U3: footprint TO_SOT_Packages_SMD:SOT-23-5 -> LibreSolar:SOT-23-5; symbol AP2210-3.3 -> LibreSolar:AP2210-3.3
Connections:
- wire segments 51 -> 69
Changed lines of the file:
@@
-EESchema Schematic File Version 2
-LIBS:IEC-60617
-LIBS:LibreSolar
-LIBS:power
-LIBS:device
-LIBS:conn
-LIBS:logo
+EESchema Schematic File Version 4
 LIBS:BMS-5s-cache
 EELAYER 26 0
@@
 $EndDescr
 $Comp
-L GND #PWR017
+L power:GND #PWR017
 U 1 1 58C300D5
 P 4000 5600
@@
 $EndComp
 $Comp
-L GND #PWR018
+L power:GND #PWR018
 U 1 1 58C300DB
 P 3600 5600
@@
 $EndComp
 $Comp
-L GND #PWR019
+L power:GND #PWR019
 U 1 1 58C300E7
 P 2300 5600
@@
 $EndComp
 $Comp
-L GND #PWR020
+L power:GND #PWR020
 U 1 1 58C300ED
 P 8200 3100
@@
 $EndComp
 $Comp
-L GND #PWR021
+L power:GND #PWR021
 U 1 1 58C300F3
 P 7900 3100
@@
 $EndComp
 $Comp
-L GND #PWR022
+L power:GND #PWR022
 U 1 1 58C300F9
 P 7100 3100
@@
 $EndComp
 $Comp
-L GND #PWR023
+L power:GND #PWR023
 U 1 1 58C30100
 P 6100 2700
@@
 $EndComp
 $Comp
-L GND #PWR024
+L power:GND #PWR024
 U 1 1 58C30106
 P 3800 2600
@@
 $EndComp
 $Comp
-L GND #PWR025
+L power:GND #PWR025
 U 1 1 58C3010C
 P 4800 2600
@@
 $EndComp
 $Comp
-L GND #PWR026
+L power:GND #PWR026
 U 1 1 58C30112
 P 3200 2600
@@
 $EndComp
 $Comp
-L +3.3V #PWR027
+L power:+3.3V #PWR027
 U 1 1 58C30118
 P 4000 4900
@@
 $EndComp
 $Comp
-L R R28
+L Project:R R28
 U 1 1 58C3011E
 P 7100 2900
@@
 $EndComp
 $Comp
-L +5V #PWR028
+L power:+5V #PWR028
 U 1 1 58C30125
 P 8200 2200
@@
 $EndComp
 $Comp
-L D D13
+L Project:D D13
 U 1 1 58C3012C
 P 6800 1700
@@
 $EndComp
 $Comp
-L C C21
+L Project:C C21
 U 1 1 58C30133
 P 2300 5300
@@
 F 0 "C21" H 2325 5375 50  0000 L CNN
 F 1 "1u" H 2325 5225 50  0000 L CNN
-F 2 "LibreSolar:C_0603_1608" H 2300 5100 50  0001 C CNN
+F 2 "LibreSolar:C_0805_2012" H 2300 5100 50  0001 C CNN
 F 3 "" H 2325 5375 50  0000 C CNN
-F 4 "Murata" H -5700 2550 50  0001 C CNN "Manufacturer"
-F 5 "GRM188R61H105KAALD" H -5700 2550 50  0001 C CNN "PartNumber"
-F 6 "X5R" H 0   0   60  0001 C CNN "Remarks"
+F 4 "Yageo" H -5700 2550 50  0001 C CNN "Manufacturer"
+F 5 "CC0805KKX7R9BB105" H -5700 2550 50  0001 C CNN "PartNumber"
+F 6 "" H 0   0   60  0001 C CNN "Remarks"
 	1    2300 5300
 	1    0    0    -1
 $EndComp
 $Comp
-L C C20
+L Project:C C20
 U 1 1 58C3013A
 P 8200 2800
@@
 $EndComp
 $Comp
-L C C19
+L Project:C C19
 U 1 1 58C30141
 P 7900 2800
@@
 $EndComp
 $Comp
-L R R27
+L Project:R R27
 U 1 1 58C30148
 P 7100 2500
@@
 $EndComp
 $Comp
-L D_Schottky D14
+L Project:D_Schottky D14
 U 1 1 58C3014F
 P 6100 2500
 F 0 "D14" H 6100 2600 50  0000 C CNN
 F 1 "SS16FP" H 6100 2400 50  0000 C CNN
-F 2 "Diodes_SMD:D_PowerDI-123" V 6100 2500 50  0001 C CNN
+F 2 "Diode_SMD:D_PowerDI-123" V 6100 2500 50  0001 C CNN
 F 3 "" V 6100 2500 50  0000 C CNN
 F 4 "Diodes Inc." H 1400 -100 50  0001 C CNN "Manufacturer"
@@
 $EndComp
 $Comp
-L C C15
+L Project:C C15
 U 1 1 58C30156
 P 6050 2100
@@
 F 2 "LibreSolar:C_0603_1608" H 6050 2100 50  0001 C CNN
 F 3 "" H 6050 2100 50  0000 C CNN
-F 4 "Murata" H 1400 -100 50  0001 C CNN "Manufacturer"
-F 5 "GRM188R71H104KA93D" H 1400 -100 50  0001 C CNN "PartNumber"
+F 4 "Yageo" H 1400 -100 50  0001 C CNN "Manufacturer"
+F 5 "CC0603KRX7R9BB104" H 1400 -100 50  0001 C CNN "PartNumber"
 	1    6050 2100
 	0    -1   -1   0
 $EndComp
 $Comp
-L C C16
+L Project:C C16
 U 1 1 58C3015D
 P 3200 2400
@@
 F 0 "C16" H 3225 2475 50  0000 L CNN
 F 1 "1u" H 3225 2325 50  0000 L CNN
-F 2 "LibreSolar:C_0603_1608" H 3200 2200 50  0001 C CNN
+F 2 "LibreSolar:C_0805_2012" H 3200 2200 50  0001 C CNN
 F 3 "" H 3225 2475 50  0000 C CNN
-F 4 "Murata" H 3200 2400 60  0001 C CNN "Manufacturer"
-F 5 "GRM188R61H105KAALD" H 3200 2400 60  0001 C CNN "PartNumber"
-F 6 "X5R" H 0   0   60  0001 C CNN "Remarks"
+F 4 "Yageo" H 3200 2400 60  0001 C CNN "Manufacturer"
+F 5 "CC0805KKX7R9BB105" H 3200 2400 60  0001 C CNN "PartNumber"
+F 6 "" H 0   0   60  0001 C CNN "Remarks"
 	1    3200 2400
 	1    0    0    -1
 $EndComp
 $Comp
-L C C17
+L Project:C C17
 U 1 1 58C30164
 P 3800 2400
@@
 $EndComp
 $Comp
-L L L1
+L Project:L L1
 U 1 1 58C3016B
 P 3500 2100
 F 0 "L1" H 3500 2170 50  0000 C CNN
 F 1 "4.7uH" H 3500 2050 50  0000 C CNN
-F 2 "Inductors_SMD:L_0805" V 3500 2100 50  0001 C CNN
-F 3 "" V 3500 2100 50  0000 C CNN
+F 2 "Inductor_SMD:L_0805_2012Metric" H 3400 2070 50  0001 C CNN
+F 3 "" H 3500 2170 50  0001 C CNN
 F 4 "Murata" H 800 -100 50  0001 C CNN "Manufacturer"
 F 5 "LQM21PN4R7NGRD" H 800 -100 50  0001 C CNN "PartNumber"
@@
 $EndComp
 $Comp
-L C C23
+L Project:C C23
 U 1 1 58C3017A
 P 3600 5400
@@
 F 2 "LibreSolar:C_0603_1608" H 3600 5200 50  0001 C CNN
 F 3 "" H 3625 5475 50  0000 C CNN
-F 4 "Murata" H -5750 2600 50  0001 C CNN "Manufacturer"
-F 5 "GRM1885C2A101JA01D" H -5750 2600 50  0001 C CNN "PartNumber"
+F 4 "Yageo" H -5750 2600 50  0001 C CNN "Manufacturer"
+F 5 "CC0603JRNPO9BN101" H -5750 2600 50  0001 C CNN "PartNumber"
 	1    3600 5400
 	1    0    0    -1
 $EndComp
 $Comp
-L C C22
+L Project:C C22
 U 1 1 58C30181
 P 4000 5300
@@
 $EndComp
 $Comp
-L L L2
+L Project:L L2
 U 1 1 58C30191
 P 6650 2300
 F 0 "L2" H 6650 2370 50  0000 C CNN
 F 1 "22uH" H 6650 2250 50  0000 C CNN
-F 2 "LibreSolar:L_WE-TPC-4818" V 6650 2300 50  0001 C CNN
-F 3 "" V 6650 2300 50  0000 C CNN
+F 2 "LibreSolar:L_WE-TPC-4818" H 6550 2270 50  0001 C CNN
+F 3 "" H 6650 2370 50  0001 C CNN
 F 4 "Bourns" H 1375 -100 50  0001 C CNN "Manufacturer"
 F 5 "SRR4028-220Y" H 1375 -100 50  0001 C CNN "PartNumber"
@@
 $EndComp
 $Comp
-L MCP16331-CH U2
+L Project:MCP16331-CH U2
 U 1 1 58BDBD3F
 P 5300 2300
 F 0 "U2" H 5300 2650 50  0000 C CNN
 F 1 "MCP16331-CH" H 5300 1950 50  0000 C CNN
-F 2 "TO_SOT_Packages_SMD:SOT-23-6" H 5300 1850 50  0001 C CNN
+F 2 "LibreSolar:SOT-23-6" H 5300 1850 50  0001 C CNN
 F 3 "" H 4900 2700 50  0000 C CNN
 F 4 "Microchip" H 1400 -50 50  0001 C CNN "Manufacturer"
@@
 $EndComp
 $Comp
-L AP2210-3.3 U3
+L LibreSolar:AP2210-3.3 U3
 U 1 1 58BDC485
 P 3100 5200
 F 0 "U3" H 3100 5550 50  0000 C CNN
 F 1 "AP2210-3.3" H 3100 4850 50  0000 C CNN
-F 2 "TO_SOT_Packages_SMD:SOT-23-5" H 3100 4700 50  0001 C CNN
+F 2 "LibreSolar:SOT-23-5" H 3100 4700 50  0001 C CNN
 F 3 "" H 3100 5200 50  0000 C CNN
 F 4 "Diodes Inc." H -5750 2650 50  0001 C CNN "Manufacturer"
@@
 $EndComp
 $Comp
-L GND #PWR029
+L power:GND #PWR029
 U 1 1 58BDC73F
 P 2600 5600
@@
 $EndComp
 $Comp
-L +5V #PWR030
+L power:+5V #PWR030
 U 1 1 58BDCD2C
 P 2300 4900
@@
 $EndComp
 $Comp
-L PWR_FLAG #FLG031
+L power:PWR_FLAG #FLG031
 U 1 1 58BFEDCA
 P 7400 2200
@@
 $EndComp
 $Comp
-L PWR_FLAG #FLG032
+L power:PWR_FLAG #FLG032
 U 1 1 58BFEEDA
 P 4300 2000
@@
 BAT+
 Wire Wire Line
-	3500 5000 4000 5000
-Wire Wire Line
-	4000 4900 4000 5200
-Wire Wire Line
-	6750 2300 8200 2300
-Wire Wire Line
-	2300 5000 2700 5000
+	3500 5000 3600 5000
+Wire Wire Line
+	4000 4900 4000 5000
+Wire Wire Line
+	6750 2300 7100 2300
+Wire Wire Line
+	2300 5000 2600 5000
 Wire Wire Line
 	7100 2300 7100 2400
 Wire Wire Line
-	2300 4900 2300 5200
+	2300 4900 2300 5000
 Wire Wire Line
 	7200 1700 7200 2300
@@
 	3600 5500 3600 5600
 Wire Wire Line
-	7100 2600 7100 2800
+	7100 2600 7100 2700
 Wire Wire Line
 	5700 2500 5800 2500
@@
 	5800 2500 5800 2900
 Wire Wire Line
-	5700 2100 5950 2100
+	5700 2100 5800 2100
 Wire Wire Line
 	5800 1700 5800 2100
 Wire Wire Line
-	5700 2300 6550 2300
+	5700 2300 6100 2300
 Wire Wire Line
 	6100 2400 6100 2300
@@
 	6300 2100 6300 2300
 Wire Wire Line
-	3600 2100 4900 2100
+	3600 2100 3800 2100
 Wire Wire Line
 	3800 2300 3800 2100
@@
 	4900 2300 4800 2300
 Wire Wire Line
-	8200 2200 8200 2700
+	8200 2200 8200 2300
 Wire Wire Line
 	4800 2500 4900 2500
@@
 	4300 2000 4300 2100
 Wire Wire Line
-	2900 2100 3400 2100
+	2900 2100 3200 2100
 Connection ~ 4000 5000
 Connection ~ 7100 2300
@@
 5V to 3.3V (LDO)
 $Comp
-L GND #PWR033
+L power:GND #PWR033
 U 1 1 58CE7EFC
 P 4100 2600
@@
 $EndComp
 $Comp
-L C C18
+L Project:C C18
 U 1 1 58CE7F0D
 P 4100 2400
@@
 F 2 "LibreSolar:C_0603_1608" H 4100 2200 50  0001 C CNN
 F 3 "" H 4125 2475 50  0000 C CNN
-F 4 "Murata" H 4100 2400 60  0001 C CNN "Manufacturer"
-F 5 "GRM188R71H104KA93D" H 4100 2400 60  0001 C CNN "PartNumber"
+F 4 "Yageo" H 4100 2400 60  0001 C CNN "Manufacturer"
+F 5 "CC0603KRX7R9BB104" H 4100 2400 60  0001 C CNN "PartNumber"
 	1    4100 2400
 	1    0    0    -1
@@
 PWR_EN
 $Comp
-L TEST TP2
+L Connector:Test_Point TP2
 U 1 1 5916EF82
 P 3600 4900
@@
 Connection ~ 3600 5000
 $Comp
-L TEST TP1
+L Connector:Test_Point TP1
 U 1 1 5916F2AF
 P 7700 2200
@@
 	7900 2700 7900 2300
 Connection ~ 7900 2300
+Wire Wire Line
+	4000 5000 4000 5200
+Wire Wire Line
+	7100 2300 7200 2300
+Wire Wire Line
+	7200 2300 7400 2300
+Wire Wire Line
+	3200 2100 3400 2100
+Wire Wire Line
+	7100 2700 7100 2800
+Wire Wire Line
+	5800 2100 5950 2100
+Wire Wire Line
+	6100 2300 6300 2300
+Wire Wire Line
+	6300 2300 6550 2300
+Wire Wire Line
+	3800 2100 4100 2100
+Wire Wire Line
+	8200 2300 8200 2700
+Wire Wire Line
+	2300 5000 2300 5200
+Wire Wire Line
+	7400 2300 7700 2300
+Wire Wire Line
+	4300 2100 4900 2100
+Wire Wire Line
+	4100 2100 4300 2100
+Wire Wire Line
+	2600 5000 2700 5000
+Wire Wire Line
+	3600 5000 4000 5000
+Wire Wire Line
+	7700 2300 7900 2300
+Wire Wire Line
+	7900 2300 8200 2300
 $EndSCHEMATC

Commit message: Diode part number corrected, closing issue #9
Parts:
- D13: value 1N4148W-7-F -> 1N4148WS-7-F; PartNumber 1N4148W-7-F -> 1N4148WS-7-F
Changed lines of the file:
@@
 P 6800 1700
 F 0 "D13" H 6800 1800 50  0000 C CNN
-F 1 "1N4148W-7-F" H 6800 1600 50  0000 C CNN
+F 1 "1N4148WS-7-F" H 6800 1600 50  0000 C CNN
 F 2 "LibreSolar:D_SOD-323" H 6800 1700 50  0001 C CNN
 F 3 "" H 6800 1700 50  0001 C CNN
 F 4 "Diodes Inc." H 1425 -100 50  0001 C CNN "Manufacturer"
-F 5 "1N4148W-7-F" H 1425 -100 50  0001 C CNN "PartNumber"
+F 5 "1N4148WS-7-F" H 1425 -100 50  0001 C CNN "PartNumber"
 	1    6800 1700
 	1    0    0    -1
